Commit message: Update robot_proyecto.xacro

File: urdf/robot_proyecto.xacro (robot description, xacro)
@@ -170,15 +170,17 @@
   <axis xyz="0.0 1.0 0.0"/>
 </joint>
-<joint name="Revolucion2" type="continuous">
+<joint name="Revolucion2" type="revolute">
   <origin xyz="0.0 0.5 0.0" rpy="0 0 0"/>
   <parent link="rot2_1"/>
   <child link="rot3_1"/>
   <axis xyz="-1.0 0.0 0.0"/>
-</joint>
-<joint name="Revolucion3" type="continuous">
+  <limit upper="2.7" lower="-2.7" effort="100" velocity="100"/>
+</joint>
+<joint name="Revolucion3" type="revolute">
   <origin xyz="0.13 0.000627 0.2" rpy="0 0 0"/>
   <parent link="rot1_1"/>
   <child link="rot2_1"/>
   <axis xyz="1.0 0.0 0.0"/>
+  <limit upper="4.14" lower="-1.0" effort="100" velocity="100"/>
 </joint>
 <joint name="Revolucion4" type="continuous">
@@ -193,5 +195,5 @@
   <child link="slider3_1"/>
   <axis xyz="0.0 0.0 1.0"/>
-  <limit upper="0.0" lower="0.0" effort="100" velocity="100"/>
+  <limit upper="0.48" lower="0.0" effort="100" velocity="100"/>
 </joint>
 <joint name="Corredera6" type="prismatic">
@@ -200,5 +202,5 @@
   <child link="slider2_1"/>
   <axis xyz="1.0 0.0 0.0"/>
-  <limit upper="0.0" lower="0.0" effort="100" velocity="100"/>
+  <limit upper="0.85" lower="-0.85" effort="100" velocity="100"/>
 </joint>
 <joint name="Corredera7" type="prismatic">
@@ -207,5 +209,5 @@
   <child link="slider1_1"/>
   <axis xyz="0.0 1.0 0.0"/>
-  <limit upper="0.0" lower="0.0" effort="100" velocity="100"/>
+  <limit upper="0.9" lower="-0.9" effort="100" velocity="100"/>
 </joint>
 </robot>

Commit message: Update robot_proyecto.xacro

File: urdf/robot_proyecto.xacro (robot description, xacro)
@@ -15,5 +15,5 @@
       <mesh filename="package://robot_proyecto_description/meshes/base_link.stl" scale="0.001 0.001 0.001"/>
     </geometry>
-    <material name="silver"/>
+    <material name="white"/>
   </visual>
   <collision>
@@ -35,5 +35,5 @@
       <mesh filename="package://robot_proyecto_description/meshes/rot4_1.stl" scale="0.001 0.001 0.001"/>
     </geometry>
-    <material name="silver"/>
+    <material name="yellow"/>
   </visual>
   <collision>
@@ -55,5 +55,5 @@
       <mesh filename="package://robot_proyecto_description/meshes/rot3_1.stl" scale="0.001 0.001 0.001"/>
     </geometry>
-    <material name="silver"/>
+    <material name="red"/>
   </visual>
   <collision>
@@ -75,5 +75,5 @@
       <mesh filename="package://robot_proyecto_description/meshes/rot2_1.stl" scale="0.001 0.001 0.001"/>
     </geometry>
-    <material name="silver"/>
+    <material name="blue"/>
   </visual>
   <collision>
@@ -95,5 +95,5 @@
       <mesh filename="package://robot_proyecto_description/meshes/rot1_1.stl" scale="0.001 0.001 0.001"/>
     </geometry>
-    <material name="silver"/>
+    <material name="red"/>
   </visual>
   <collision>
@@ -135,5 +135,5 @@
       <mesh filename="package://robot_proyecto_description/meshes/slider2_1.stl" scale="0.001 0.001 0.001"/>
     </geometry>
-    <material name="silver"/>
+    <material name="green"/>
   </visual>
   <collision>
@@ -155,5 +155,5 @@
       <mesh filename="package://robot_proyecto_description/meshes/slider1_1.stl" scale="0.001 0.001 0.001"/>
     </geometry>
-    <material name="silver"/>
+    <material name="yellow"/>
   </visual>
   <collision>
